File: z80badgev2/z80badgev2.kicad_pcb (KiCad board)
At the start: 2 copper layers, 81.9 x 93.6 mm, 29 parts, among them J2 Conn_01x20_Pin, J3 Conn_01x20_Pin, SW1 Reset, SW10 Input, SW11 Input, SW2 Input, SW3 Input, SW4 Bus Release, SW5 Power, SW6 Input, SW7 Input, SW8 Input, SW9 Input, U1 Z84C0010P, U2 Z84C20, U3 28C256 SOP28, U4 HM 62256 SOP28, U5 74AHCT1G32, U6 74AHCT1G04, U7 74AHCT1G32, Y1 ACO-xxxMHz

Commit message: Add files via upload
Other:
- board size 81.9 x 93.6 mm -> 81.9 x 99.4 mm
- board text added: "___ ___ _| \__/ |_ A10 |_|40 1|_| A11 A9 |_|39 2|_| A12 A8 |_|38 3|_| A13 A7 |_|37 4|_| A14 A6 |_|36 5|_| A15 A5 |_|35 6|_| CLK A4 |_|34 7|_| D4 A3 |_|33 8|_| D3 A2 |_|32 9|_| D5 A1 |_|31 10|_| D6 A0 |_|30 11|_| VCC GND |_|29 12|_| D2 ~{RFSH} |_|28 13|_| D7 ~{M1} |_|27 14|_| D0 ~{RESET} |_|26 15|_| D1 ~{BUSRQ} |_|25 16|_| ~{INT} ~{WAIT} |_|24 17|_| ~{NMI} ~{BUSAK} |_|23 18|_| ~{HALT} ~{WR} |_|22 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"
- board text added: "__________.__.__ __________ ______ _______ \____ /|__| | ____ ____\____ // __ \\ _ \ / / | | | / _ \ / ___\ / / > </ /_\ \ / /_ | | |_( <_> ) /_/ > /_/ -- \ \_/ \ /_______ \|__|____/\____/\___ /_______ \______ /\_____ / \/ /_____/ \/ \/ \/"

Commit message: Add files via upload
Other:
- outline, holes or cut-outs redrawn
- board text added: "#GADGETMARKET"
