File: z80badgev2/z80badgev2.kicad_pcb (KiCad board)
At the start: 2 copper layers, 81.9 x 99.4 mm, 29 parts, among them J2 Conn_01x20_Pin, J3 Conn_01x20_Pin, SW1 Reset, SW10 Input, SW11 Input, SW2 Input, SW3 Input, SW4 Bus Release, SW5 Power, SW6 Input, SW7 Input, SW8 Input, SW9 Input, U1 Z84C0010P, U2 Z84C20, U3 28C256 SOP28, U4 HM 62256 SOP28, U5 74AHCT1G32, U6 74AHCT1G04, U7 74AHCT1G32, Y1 ACO-xxxMHz

Commit message: Add files via upload
Parts:
- added C1: C, Capacitor_SMD:C_0805_2012Metric, F.Cu at (487.6, -9.80)
- added C2: C, Capacitor_SMD:C_0805_2012Metric, F.Cu at (431.5, -23.4)
- added C3: C, Capacitor_SMD:C_0805_2012Metric, F.Cu at (498.8, -46.8)
- added C4: C, Capacitor_SMD:C_0805_2012Metric, F.Cu at (474.0, -46.9)
- added C5: C, Capacitor_SMD:C_0805_2012Metric, B.Cu at (453.8, -22.8)
- moved U5 3.67 mm to (485.7, -58.1)
- moved U6 3.67 mm to (466.6, -62.5)
- moved U7 3.67 mm to (466.5, -58.1)
Routing:
- net /Power: track 327.6 -> 360.5 mm, vias 2 -> 4
- net GND: track 40.2 -> 56.7 mm, vias 216 -> 329
- net +5V: track 141.9 -> 152.2 mm, vias 1 -> 2
- net /~{INT}: track 88.5 -> 80.3 mm
- net /~{WR}: track 58.1 -> 64.3 mm
- net /A13: track 107.7 -> 113.5 mm
- net /A8: track 100.0 -> 105.3 mm
- net /A9: track 102.1 -> 106.9 mm
- net /A15: track 140.1 -> 144.8 mm
- net /A14: track 104.5 -> 109.1 mm
- net /A11: track 106.8 -> 111.2 mm
- net /~{RD}: track 102.4 -> 106.7 mm
- net /A12: track 99.6 -> 103.7 mm
- net /~{MREQ}: track 52.8 -> 56.5 mm
- net Net-(U4-~{CS}): track 6.36 -> 10.0 mm
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