File: z80badgev2/z80badgev2_BACKUP.kicad_pcb (KiCad board)
At the start: 2 copper layers, 81.9 x 99.4 mm, 29 parts, among them J2 Conn_01x20_Pin, J3 Conn_01x20_Pin, SW1 Reset, SW10 Input, SW11 Input, SW2 Input, SW3 Input, SW4 Bus Release, SW5 Power, SW6 Input, SW7 Input, SW8 Input, SW9 Input, U1 Z84C0010P, U2 Z84C20, U3 28C256 SOP28, U4 HM 62256 SOP28, U5 74AHCT1G32, U6 74AHCT1G04, U7 74AHCT1G32, Y1 ACO-xxxMHz

Commit message: Add files via upload
Routing:
- net GND: track 40.2 -> 305.1 mm, vias 216 -> 4
- net /~{INT}: track 88.5 -> 83.3 mm
- net /~{M1}: track 177.8 -> 179.4 mm
- net /~{BUSREQ}: track 57.7 -> 56.7 mm
- net /D5: track 117.1 -> 116.3 mm
- net /D4: track 120.7 -> 119.9 mm
- net /D3: track 117.0 -> 116.2 mm
- net /Power: track 327.6 -> 327.0 mm
